Commit message: change imu from wheeltec n100 mini to LINS358

File: src/cartographer_config/urdf/my_robot.urdf (robot description, URDF)
Before this commit: robot cartographer_backpack_3d, 3 links, 2 joints
Links:
- removed link gyro_link
- added link imu_link; visual box size=0.036 0.035 0.018
Joints:
- joint imu_link_joint: child gyro_link -> imu_link; origin xyz=0.005 0.000 0.048 rpy=3.1415926 0 1.48353 -> xyz=0.000 0.000 0.056 rpy=0 0 1.5707963
